File: esp_dock/_saved_esp_dock.sch (KiCad schematic (older format))
At the start: 10 parts, among them P1 POWER, P2 LIGHT, P3 ESP, P4 SERIAL, P5 Pgrm, SW1 Switch_SPDT_x2, U1 LM3671

Commit message: Finished v1
Changed lines of the file:
@@
 F 0 "P3" H 7900 3950 50  0000 C CNN
 F 1 "ESP" H 7900 3450 50  0000 C CNN
-F 2 "Pin_Headers:Pin_Header_Straight_2x04" H 7900 2500 50  0000 C CNN
+F 2 "Pin_Headers:Pin_Header_Straight_2x04" H 7500 3150 50  0000 C CNN
 F 3 "" H 7900 2500 50  0000 C CNN
 	1    7900 3700
