File: esp_dock/esp_dock.kicad_pcb (KiCad board)
At the start: 2 copper layers, 26.7 x 35.6 mm, 10 parts, among them P1 POWER, P2 LIGHT, P3 ESP, P4 SERIAL, P5 PRG_JMPR, SW1 Switch_SPDT_x2, U1 LM3671

Commit message: Finished v1
Parts:
- P5: value PRG_JMPR -> Pgrm; footprint Pin_Headers:Pin_Header_Straight_1x02_Pitch2.00mm -> Pin_Headers:Pin_Header_Straight_1x03_Pitch2.00mm
- moved C2 14.2 mm to (129.5, 154.9), turned to 0 degrees
- moved L1 12.8 mm to (129.5, 146.3), turned to 180 degrees
- moved C1 10.5 mm to (129.5, 148.6)
- moved P1 1.91 mm to (139.1, 150.5), turned to 0 degrees
- moved U1 0.64 mm to (129.5, 151.8), turned to 270 degrees
- moved P4 0.13 mm to (132.1, 127.5)
- moved P5 0.13 mm to (147.3, 131.6)
Connections:
- P2 pad 1: Net-(C1-Pad2) -> Net-(C1-Pad1)
- P2 pad 4: Net-(C1-Pad1) -> Net-(C1-Pad2)
- P3 pad 1: Net-(C1-Pad2) -> Net-(P3-Pad1)
- P3 pad 2: Net-(P3-Pad2) -> Net-(C2-Pad1)
- P3 pad 3: Net-(P2-Pad2) -> Net-(P2-Pad3)
- P3 pad 4: Net-(C2-Pad1) -> Net-(P3-Pad4)
- P3 pad 5: Net-(P2-Pad3) -> Net-(P2-Pad2)
- P3 pad 6: Net-(P3-Pad6) -> Net-(C2-Pad1)
- P3 pad 7: Net-(P3-Pad7) -> Net-(C1-Pad2)
- P3 pad 8: Net-(C2-Pad1) -> Net-(P3-Pad8)
- P4 pad 2: Net-(P3-Pad2) -> Net-(P3-Pad8)
- P4 pad 3: Net-(P3-Pad7) -> Net-(P3-Pad1)
- P5 pad 2: Net-(P3-Pad6) -> Net-(P3-Pad4)
Routing:
- net Net-(C1-Pad2): track 0.00 -> 70.8 mm, vias 0 -> 1
- net Net-(C2-Pad1): track 0.00 -> 59.4 mm, vias 0 -> 1
- net Net-(C1-Pad1): track 0.00 -> 54.3 mm, vias 0 -> 1
- net Net-(P3-Pad8): track 0.00 -> 31.5 mm
- net Net-(P3-Pad1): track 0.00 -> 19.9 mm
- net Net-(P2-Pad2): track 0.00 -> 19.0 mm, vias 0 -> 1
- net Net-(P2-Pad3): track 0.00 -> 14.0 mm, vias 0 -> 1
- net Net-(P3-Pad4): track 0.00 -> 13.9 mm
- net Net-(L1-Pad1): track 0.00 -> 9.97 mm, vias 0 -> 2
- net Net-(P1-Pad1): track 0.00 -> 5.98 mm
Other:
- net class Default: clearance 0.2 -> 0.1524; trace_width 0.25 -> 0.1524; via_dia 0.6 -> 0.6858; via_drill 0.4 -> 0.3302
- rule trace_clearance: 0.2 -> 0.1524
- rule trace_min: 0.2 -> 0.1524
- rule via_min_drill: 0.3 -> 0.3302
- rule via_min_size: 0.4 -> 0.6858
- board text added: "+"
- board text added: "-"
- board text added: "CI"
- board text added: "DI"
- board text added: "ESP-01"
- board text added: "GND"
- board text added: "Mode"
- board text added: "Pgrm"
- board text added: "Power"
- board text added: "Power Switch"
- board text added: "RX"
- board text added: "Raver Endpoint v1.0 Copyright (c) Bryan Hughes"
- board text added: "Run"
- board text added: "Serial"
- board text added: "TX"
- board text added: "VCC"

Commit message: Finished v1.5 of the board
Parts:
- C1, C2, L1, U1: moved to B.Cu
- moved C2 19.8 mm to (142.9, 140.3)
- moved U1 14.5 mm to (142.9, 146.1), turned to 0 degrees
- moved L1 13.8 mm to (142.9, 142.9)
- moved P2 12.9 mm to (138.3, 144.8), turned to 180 degrees
- moved C1 7.65 mm to (137.2, 148.0), turned to 180 degrees
- moved P4 5.57 mm to (135.3, 132.1), turned to 90 degrees
- moved P1 1.27 mm to (137.8, 150.5)
- moved P5 0.81 mm to (146.7, 132.1), turned to 270 degrees
- moved SW1 0.63 mm to (144.1, 149.9)
Routing:
- net Net-(C2-Pad1): track 59.4 -> 27.7 mm, vias 1 -> 0
- net Net-(C1-Pad1): track 54.3 -> 25.1 mm, vias 1 -> 0
- net Net-(P3-Pad8): track 31.5 -> 20.5 mm
- net Net-(P2-Pad2): track 19.0 -> 9.02 mm, vias 1 -> 0
- net Net-(P3-Pad1): track 19.9 -> 10.2 mm
- net Net-(C1-Pad2): track 70.8 -> 79.8 mm, vias 1 -> 0
- net Net-(P2-Pad3): track 14.0 -> 9.02 mm, vias 1 -> 0
- net Net-(L1-Pad1): track 9.97 -> 5.64 mm, vias 2 -> 0
- net Net-(P3-Pad4): track 13.9 -> 16.0 mm
- net Net-(P1-Pad1): track 5.98 -> 6.61 mm
Other:
- board size 26.7 x 35.6 mm -> 24.1 x 25.5 mm
- board text added: "PGM"
- board text added: "RUN"
- board text added: "Raver Lights Endpoint v1.5 Copyright Bryan Hughes 2016"
- board text removed: "Mode"
- board text removed: "Pgrm"
- board text removed: "Raver Endpoint v1.0 Copyright (c) Bryan Hughes"
- board text removed: "Run"
- board text removed: "Serial"

Commit message: Last minute updates
Parts:
- moved P1 1.27 mm to (139.1, 150.5)
Routing:
- net Net-(P1-Pad1): track 6.61 -> 5.34 mm
- net Net-(C1-Pad2): track 79.8 -> 81.1 mm
Other:
- board size 24.1 x 25.5 mm -> 24.1 x 25.4 mm
Changed lines of the file:
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@@
     (links 23)
     (no_connects 0)
-    (area 118.986172 121.209999 159.635972 160.3124)
+    (area 127.475599 116.525409 158.881972 155.992162)
     (thickness 1.6)
-    (drawings 29)
+    (drawings 30)
     (tracks 83)
     (zones 0)
@@
   )
   (setup
-    (last_trace_width 0.6096)
+    (last_trace_width 0.1524)
     (user_trace_width 0.1524)
     (user_trace_width 0.3048)
@@
   )
   (module Pin_Headers:Pin_Header_Straight_1x02_Pitch2.00mm (layer F.Cu)
-    (at 137.795 150.495)
+    (at 139.065 150.495)
     (descr "Through hole pin header, 1x02, 2.00mm pitch, single row")
     (tags "pin header single row")
@@
     )
   )
-  (gr_line (start 127.635 155.575) (end 127.635 155.702) (angle 90) (layer Edge.Cuts) (width 0.15))
-  (gr_line (start 151.765 155.575) (end 127.635 155.575) (angle 90) (layer Edge.Cuts) (width 0.15))
+  (gr_line (start 127.635 147.955) (end 127.635 130.175) (angle 90) (layer Edge.Cuts) (width 0.15))
+  (gr_line (start 130.81 147.955) (end 127.635 147.955) (angle 90) (layer Edge.Cuts) (width 0.15))
+  (gr_line (start 130.81 155.575) (end 130.81 147.955) (angle 90) (layer Edge.Cuts) (width 0.15))
+  (gr_line (start 151.765 155.575) (end 130.81 155.575) (angle 90) (layer Edge.Cuts) (width 0.15))
   (gr_line (start 151.638 130.175) (end 127.635 130.175) (angle 90) (layer Edge.Cuts) (width 0.15))
   (gr_text RX (at 132.715 132.08 270) (layer F.SilkS)
@@
   )
   (gr_line (start 151.765 130.175) (end 151.765 155.575) (angle 90) (layer Edge.Cuts) (width 0.15))
-  (gr_line (start 127.635 130.175) (end 127.635 155.575) (angle 90) (layer Edge.Cuts) (width 0.15))
   (gr_text GND (at 128.905 137.16 90) (layer B.SilkS)
     (effects (font (size 1.016 1.016) (thickness 0.1524)) (justify mirror))
@@
     (effects (font (size 1.016 1.016) (thickness 0.1524)) (justify mirror))
   )
-  (gr_text "Raver Lights Endpoint v1.5\nCopyright Bryan Hughes 2016" (at 132.334 142.24 90) (layer B.SilkS)
+  (gr_text "Raver Lights Endpoint v1.5\nCopyright Bryan Hughes 2016" (at 132.715 142.24 90) (layer B.SilkS)
     (effects (font (size 1.016 1.016) (thickness 0.1524)) (justify mirror))
   )
-  (gr_text Power (at 132.715 151.765 90) (layer F.SilkS)
+  (gr_text Power (at 133.985 151.765 90) (layer F.SilkS)
     (effects (font (size 1.016 1.016) (thickness 0.1524)))
   )
@@
     (effects (font (size 1.016 1.016) (thickness 0.1524)))
   )
-  (gr_text - (at 135.001 153.543) (layer F.SilkS)
+  (gr_text - (at 133.985 154.305) (layer F.SilkS)
     (effects (font (size 1.5 1.5) (thickness 0.1524)))
   )
-  (gr_text + (at 135.001 149.606) (layer F.SilkS)
+  (gr_text + (at 133.985 148.59) (layer F.SilkS)
     (effects (font (size 1.5 1.5) (thickness 0.1524)))
   )
-  (gr_line (start 139.7 154.94) (end 139.7 147.955) (angle 90) (layer F.SilkS) (width 0.2))
-  (gr_line (start 131.445 154.94) (end 139.7 154.94) (angle 90) (layer F.SilkS) (width 0.2))
-  (gr_line (start 131.445 147.955) (end 131.445 154.94) (angle 90) (layer F.SilkS) (width 0.2))
+  (gr_line (start 140.97 154.94) (end 140.97 147.955) (angle 90) (layer F.SilkS) (width 0.2))
+  (gr_line (start 132.715 154.94) (end 140.97 154.94) (angle 90) (layer F.SilkS) (width 0.2))
+  (gr_line (start 132.715 147.955) (end 132.715 154.94) (angle 90) (layer F.SilkS) (width 0.2))
   (gr_line (start 141.605 149.86) (end 142.24 149.86) (angle 90) (layer F.SilkS) (width 0.2))
   (gr_line (start 141.605 155.575) (end 141.605 149.86) (angle 90) (layer F.SilkS) (width 0.2))
@@
   (segment (start 138.303 144.78) (end 138.303 147.848) (width 0.6096) (layer B.Cu) (net 1))
   (segment (start 138.303 147.848) (end 138.41 147.955) (width 0.6096) (layer B.Cu) (net 1))
-  (segment (start 137.795 152.495) (end 149.765 152.495) (width 0.6096) (layer F.Cu) (net 2))
+  (segment (start 139.065 152.495) (end 149.765 152.495) (width 0.6096) (layer F.Cu) (net 2) (status 10))
   (segment (start 151.257 148.717) (end 147.32 144.78) (width 0.6096) (layer F.Cu) (net 2))
   (segment (start 151.257 151.003) (end 151.257 148.717) (width 0.6096) (layer F.Cu) (net 2))
@@
   (segment (start 139.954 145.542) (end 140.462 146.05) (width 0.6096) (layer B.Cu) (net 2))
   (segment (start 139.954 138.176) (end 139.954 145.542) (width 0.6096) (layer B.Cu) (net 2))
-  (segment (start 137.795 152.495) (end 136.62 152.495) (width 1.2192) (layer F.Cu) (net 2))
+  (segment (start 139.065 152.495) (end 136.62 152.495) (width 1.2192) (layer F.Cu) (net 2) (status 10))
   (segment (start 135.89 151.765) (end 135.89 138.43) (width 1.2192) (layer F.Cu) (net 2))
   (segment (start 136.62 152.495) (end 135.89 151.765) (width 1.2192) (layer F.Cu) (net 2))
-  (segment (start 137.795 152.495) (end 136.62 152.495) (width 0.6096) (layer B.Cu) (net 2))
+  (segment (start 139.065 152.495) (end 136.62 152.495) (width 0.6096) (layer B.Cu) (net 2) (status 10))
   (segment (start 135.91 151.785) (end 135.91 147.955) (width 0.6096) (layer B.Cu) (net 2))
   (segment (start 136.62 152.495) (end 135.91 151.785) (width 0.6096) (layer B.Cu) (net 2))
@@
   (segment (start 147.32 142.24) (end 138.303 142.24) (width 0.3048) (layer F.Cu) (net 5))
   (segment (start 138.303 139.7) (end 147.32 139.7) (width 0.3048) (layer F.Cu) (net 6))
-  (segment (start 137.795 150.495) (end 143.51 150.495) (width 1.2192) (layer F.Cu) (net 7))
+  (segment (start 139.065 150.495) (end 143.51 150.495) (width 1.2192) (layer F.Cu) (net 7) (status 10))
   (segment (start 143.51 150.495) (end 144.145 149.86) (width 1.2192) (layer F.Cu) (net 7))
   (segment (start 139.255 132.08) (end 140.97 132.08) (width 0.3048) (layer F.Cu) (net 9))
