File: coordinator_board/Coordinator Board.sch (KiCad schematic (older format))
At the start: 19 parts, among them P1 POWER, P10 Mounting Hole, P11 Mounting Hole, P12 Mounting Hole, P13 Mounting Hole, P3 Peripheral, P4 SERIAL, P5 PGRM, SW1 Switch_SPDT_x2, U1 LM3671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

Commit message: Added rotary encoder to schematic
Connections:
- wire segments 91 -> 70
Changed lines of the file:
@@
 	3850 2950 4000 2950
 Wire Wire Line
-	3000 3150 3000 3500
-Wire Wire Line
-	3000 3500 3000 3600
+	3000 3150 3000 3600
 Wire Wire Line
 	3000 3500 3050 3500
 Connection ~ 3000 3500
 Wire Wire Line
-	2700 3700 2850 3700
+	2700 3700 3050 3700
 Wire Wire Line
-	2850 3700 3050 3700
+	2850 3550 2850 4450
 Wire Wire Line
-	2850 3550 2850 3700
-Wire Wire Line
-	2850 3700 2850 4450
-Wire Wire Line
-	2850 4450 4850 4450
-Wire Wire Line
-	4850 4450 5350 4450
-Wire Wire Line
-	5350 4450 6650 4450
-Wire Wire Line
-	6650 4450 8050 4450
-Wire Wire Line
-	8050 4450 8750 4450
+	2850 4450 8750 4450
 Connection ~ 2850 3700
 Wire Wire Line
@@
 	4000 3150 4000 2950
 Wire Wire Line
-	2850 3150 3000 3150
-Wire Wire Line
-	3000 3150 4000 3150
+	2850 3150 4000 3150
 Wire Wire Line
 	2850 3150 2850 3250
 Connection ~ 3000 3150
 Wire Wire Line
-	4850 2450 4850 3350
-Wire Wire Line
-	4850 3350 4850 3500
-Wire Wire Line
-	4850 3500 4850 3700
-Wire Wire Line
-	4850 3700 4850 3850
+	4850 2450 4850 3850
 Wire Wire Line
 	3850 3700 4850 3700
@@
 Connection ~ 4850 3500
 Wire Wire Line
-	5350 3050 5350 4450
-Wire Wire Line
-	5350 4450 5350 4550
+	5350 3050 5350 4550
 Connection ~ 5350 4450
 Wire Wire Line
@@
 	8650 3750 8550 3750
 Wire Wire Line
-	4850 2450 5750 2450
-Wire Wire Line
-	5750 2450 6650 2450
-Wire Wire Line
-	6650 2450 8650 2450
-Wire Wire Line
-	8650 2450 9050 2450
+	4850 2450 9050 2450
 Connection ~ 8650 3050
 Connection ~ 4850 3350
@@
 Connection ~ 6650 2450
 Wire Wire Line
-	6650 2850 6650 2950
-Wire Wire Line
-	6650 2950 6650 3350
+	6650 2850 6650 3350
 Wire Wire Line
 	6300 2850 6300 3050
@@
 	5750 3250 5950 3250
 Wire Wire Line
-	5750 2450 5750 3250
-Wire Wire Line
-	5750 3250 5750 4350
+	5750 2450 5750 4350
 Connection ~ 5750 2450
 Wire Wire Line
-	5350 3050 6300 3050
-Wire Wire Line
-	6300 3050 6750 3050
+	5350 3050 6750 3050
 Wire Wire Line
 	6750 3250 6250 3250
 Wire Wire Line
-	8650 2450 8650 3050
-Wire Wire Line
-	8650 3050 8650 3750
+	8650 2450 8650 3750
 Wire Wire Line
 	8550 3050 8650 3050
@@
 	8050 4450 8050 4550
 Wire Wire Line
-	5750 4350 6750 4350
-Wire Wire Line
-	6750 4350 8150 4350
+	5750 4350 8150 4350
 Connection ~ 5750 3250
 Wire Wire Line
@@
 	8750 5000 10050 5000
 Wire Wire Line
-	8750 4450 8750 4700
-Wire Wire Line
-	8750 4700 8750 5000
+	8750 4450 8750 5000
 Connection ~ 8050 4450
 Wire Wire Line

Commit message: Added rotary encoder footprint
Parts:
- removed P10, P11, P12, P13: Mounting Hole, Mounting_Holes:MountingHole_2.2mm_M2, symbol CONN_01X01
- removed P3: Peripheral, Pin_Headers:Pin_Header_Straight_1x04_Pitch2.00mm, symbol CONN_01X04
- U5: footprint (none) -> Rotary_Encoder:Rotary_Encoder
Connections:
- wire segments 70 -> 60
- no-connect marks 11 -> 10
Changed lines of the file:
@@
-$EndComp
-$Comp
-L CONN_01X04 P3
-U 1 1 589796B0
-P 8000 4750
-F 0 "P3" H 8000 5000 50  0000 C CNN
-F 1 "Peripheral" V 8100 4750 50  0000 C CNN
-F 2 "Pin_Headers:Pin_Header_Straight_1x04_Pitch2.00mm" V 8800 4800 50  0000 C CNN
-F 3 "" H 8000 4750 50  0000 C CNN
-	1    8000 4750
-	0    1    1    0
 $EndComp
 $Comp
@@
 	-1   0    0    1
 $EndComp
-$Comp
-L CONN_01X01 P10
-U 1 1 589A31E3
-P 1800 4500
-F 0 "P10" H 1800 4600 50  0000 C CNN
-F 1 "Mounting Hole" H 2150 4500 50  0000 C CNN
-F 2 "Mounting_Holes:MountingHole_2.2mm_M2" H 1800 4700 50  0000 C CNN
-F 3 "" H 1800 4500 50  0000 C CNN
-	1    1800 4500
-	1    0    0    -1
-$EndComp
-$Comp
-L CONN_01X01 P11
-U 1 1 589A324B
-P 1800 4750
-F 0 "P11" H 1800 4850 50  0000 C CNN
-F 1 "Mounting Hole" H 2150 4750 50  0000 C CNN
-F 2 "Mounting_Holes:MountingHole_2.2mm_M2" H 1800 5200 50  0000 C CNN
-F 3 "" H 1800 4750 50  0000 C CNN
-	1    1800 4750
-	1    0    0    -1
-$EndComp
-$Comp
-L CONN_01X01 P12
-U 1 1 589A32AD
-P 1800 5000
-F 0 "P12" H 1800 5100 50  0000 C CNN
-F 1 "Mounting Hole" H 2150 5000 50  0000 C CNN
-F 2 "Mounting_Holes:MountingHole_2.2mm_M2" H 1800 5700 50  0000 C CNN
-F 3 "" H 1800 5000 50  0000 C CNN
-	1    1800 5000
-	1    0    0    -1
-$EndComp
-$Comp
-L CONN_01X01 P13
-U 1 1 589A32E6
-P 1800 5250
-F 0 "P13" H 1800 5350 50  0000 C CNN
-F 1 "Mounting Hole" H 2150 5250 50  0000 C CNN
-F 2 "Mounting_Holes:MountingHole_2.2mm_M2" H 1800 6200 50  0000 C CNN
-F 3 "" H 1800 5250 50  0000 C CNN
-	1    1800 5250
-	1    0    0    -1
-$EndComp
-NoConn ~ 1600 4500
-NoConn ~ 1600 4750
-NoConn ~ 1600 5000
 NoConn ~ 1600 5250
 Wire Wire Line
@@
 	3850 3500 3900 3500
 Wire Wire Line
-	4000 3150 4000 2950
+	4000 2950 4000 3150
 Wire Wire Line
-	2850 3150 4000 3150
+	4000 3150 2850 3150
 Wire Wire Line
 	2850 3150 2850 3250
@@
 Wire Wire Line
 	8550 3050 8650 3050
-Wire Wire Line
-	8050 4450 8050 4550
-Wire Wire Line
-	5750 4350 8150 4350
 Connection ~ 5750 3250
 Wire Wire Line
-	8150 4350 8150 4550
-Wire Wire Line
-	6650 4150 7950 4150
-Wire Wire Line
-	8550 3150 8750 3150
-Wire Wire Line
-	8750 3150 8750 4250
-Wire Wire Line
-	8750 4250 7850 4250
-Wire Wire Line
 	6450 3450 6750 3450
-Wire Wire Line
-	6650 3550 6750 3550
-Wire Wire Line
-	7850 4250 7850 4550
-Wire Wire Line
-	7950 4150 7950 4550
-Wire Wire Line
-	6650 3550 6650 4150
 Wire Wire Line
 	6750 3150 6550 3150
@@
 Wire Wire Line
 	6750 4550 6750 4350
-Connection ~ 6750 4350
 Wire Wire Line
 	6650 4550 6650 4450
@@
 F 0 "U5" V 9350 4850 60  0000 C CNN
 F 1 "Rotary_Encoder" V 9750 4850 60  0000 C CNN
-F 2 "" H 9500 4850 60  0000 C CNN
+F 2 "Rotary_Encoder:Rotary_Encoder" V 9900 4850 60  0000 C CNN
 F 3 "" H 9500 4850 60  0000 C CNN
 	1    9500 4850
@@
 	10050 4800 10050 5000
 Wire Wire Line
-	8750 5000 10050 5000
+	10050 5000 8750 5000
 Wire Wire Line
-	8750 4450 8750 5000
-Connection ~ 8050 4450
+	8750 5000 8750 4450
 Wire Wire Line
 	9050 4700 8750 4700
@@
 Wire Wire Line
 	9050 2450 9050 2550
+NoConn ~ 8550 3150
+Wire Wire Line
+	6750 4350 5750 4350
+NoConn ~ 6750 3550
 $EndSCHEMATC

Commit message: Finished revision of coordinator board
Parts:
- added R3: 0, Resistors_SMD:R_0805_HandSoldering, symbol R
- added R4, R6: 10k, Resistors_SMD:R_0805_HandSoldering, symbol R
- R5: renamed from R3; footprint (none) -> Resistors_SMD:R_0805_HandSoldering
- renumbered R2 to R1, R1 to R2
Connections:
- net GND: now reaches C1.2, C2.2, P1.2 (P2), P4.3 (P3), P5.1 (P1), U1.2 (GND), U3.9 (GND), U4.2 (GND), U5.2 (C), U5.5 (GND)
- net GND: now also R4.2
- net +3V3: now reaches C2.1, L1.2, R5.2, U1.4 (FB), U3.8 (VCC), U4.1 (VCC)
- net +3V3: now also R1.1, R3.1, R6.1; no longer R1.2, R2.2, U3.1 (REST)
- net at U3.10 (GPIO15): now also R4.1; no longer U4.3 (SCL)
- net at U3.11 (GPIO2): now also R1.2; no longer R1.1
- net at U3.14 (GPIO5): now also U4.3 (SCL)
- net at U3.4 (GPIO16): now also U5.1 (A); no longer U5.3 (B)
- net at U3.5 (GPIO14): now also U5.3 (B); no longer U5.1 (A)
- new net: R6.2, U3.1 (REST)
- new net: R2.2, R3.2
- no-connect marks 10 -> 8
Other:
- moved on the sheet: P5, R1, R2, R5

Commit message: Created v2.6 of the coordinator board
Parts:
- removed R3: 0, Resistors_SMD:R_0805_HandSoldering, symbol R
- removed U5: Rotary_Encoder, Rotary_Encoder:Rotary_Encoder, symbol Rotary_Encoder
- added U5: SF303GJ26, SF303GJ26:SF303GJ26, symbol SF303GJ26
- P5: value PGRM -> PROGRAM
Connections:
- net +3V3: now also R2.2
- net GND: now also U5.5 (COM)
- net at U3.4 (GPIO16): now also U5.1 (A)
- net at U3.5 (GPIO14): now also U5.3 (C)
- net at U3.6 (GPIO12): now also U5.4 (B)
- net at U3.7 (GPIO13): now also U5.6 (D)
Changed lines of the file:
@@
 LIBS:TSWA
 LIBS:Rotary_Encoder
+LIBS:sf303gj26
 LIBS:Coordinator Board-cache
 EELAYER 25 0
@@
 $EndComp
 $Comp
-L CONN_01X02 P5
-U 1 1 58859834
-P 6050 2650
-F 0 "P5" H 6050 2800 50  0000 C CNN
-F 1 "PGRM" V 6150 2650 50  0000 C CNN
-F 2 "Pin_Headers:Pin_Header_Straight_1x02_Pitch2.00mm" V 6650 3200 50  0000 C CNN
-F 3 "" H 6050 2650 50  0000 C CNN
-	1    6050 2650
-	0    -1   -1   0
-$EndComp
-$Comp
 L R R2
 U 1 1 58978884
@@
 NoConn ~ 7900 2550
 NoConn ~ 7800 2550
-NoConn ~ 7700 2550
 NoConn ~ 7600 2550
 NoConn ~ 7500 2550
@@
 	3850 3500 3900 3500
 Wire Wire Line
-	4000 3150 4000 2950
-Wire Wire Line
-	2850 3150 4000 3150
+	4000 2950 4000 3150
+Wire Wire Line
+	4000 3150 2850 3150
 Wire Wire Line
 	2850 3150 2850 3250
@@
 Wire Wire Line
 	6000 2850 6000 3150
-Connection ~ 6000 3050
 Wire Wire Line
 	6100 2850 6100 3350
@@
 	-1   0    0    1
 $EndComp
-$Comp
-L Rotary_Encoder U5
-U 1 1 58D36C2B
-P 9500 4850
-F 0 "U5" V 9350 4850 60  0000 C CNN
-F 1 "Rotary_Encoder" V 9750 4850 60  0000 C CNN
-F 2 "Rotary_Encoder:Rotary_Encoder" V 9900 4850 60  0000 C CNN
-F 3 "" H 9500 4850 60  0000 C CNN
-	1    9500 4850
-	0    1    1    0
-$EndComp
-Wire Wire Line
-	9950 4600 10050 4600
-Wire Wire Line
-	10050 4600 10050 3250
-Wire Wire Line
-	10050 3250 8550 3250
-Wire Wire Line
-	8550 3450 8850 3450
-Wire Wire Line
-	8550 3350 8950 3350
-Wire Wire Line
-	8950 3350 8950 4800
 Wire Wire Line
 	8550 3550 9050 3550
 Wire Wire Line
 	9050 3550 9050 3100
-NoConn ~ 8550 3150
-Wire Wire Line
-	8950 4800 9050 4800
-Wire Wire Line
-	8850 3450 8850 4600
-Wire Wire Line
-	8850 4600 9050 4600
-Wire Wire Line
-	6650 2550 6650 2650
 $Comp
 L R R6
@@
 	9350 3750 9350 3100
 $Comp
-L +3.3V #PWR?
+L +3.3V #PWR01
 U 1 1 58D6E218
 P 4850 3400
-F 0 "#PWR?" H 4850 3250 50  0001 C CNN
+F 0 "#PWR01" H 4850 3250 50  0001 C CNN
 F 1 "+3.3V" H 4850 3540 50  0000 C CNN
 F 2 "" H 4850 3400 50  0000 C CNN
@@
 $EndComp
 $Comp
-L +3.3V #PWR?
+L +3.3V #PWR02
 U 1 1 58D6E2FE
 P 6300 2550
-F 0 "#PWR?" H 6300 2400 50  0001 C CNN
+F 0 "#PWR02" H 6300 2400 50  0001 C CNN
 F 1 "+3.3V" H 6300 2690 50  0000 C CNN
 F 2 "" H 6300 2550 50  0000 C CNN
@@
 $EndComp
 $Comp
-L +3.3V #PWR?
+L +3.3V #PWR03
 U 1 1 58D6E3A2
 P 6750 4350
-F 0 "#PWR?" H 6750 4200 50  0001 C CNN
+F 0 "#PWR03" H 6750 4200 50  0001 C CNN
 F 1 "+3.3V" H 6750 4490 50  0000 C CNN
 F 2 "" H 6750 4350 50  0000 C CNN
@@
 	6750 4350 6750 4550
 $Comp
-L +3.3V #PWR?
+L +3.3V #PWR04
 U 1 1 58D6E5CC
-P 6650 2150
-F 0 "#PWR?" H 6650 2000 50  0001 C CNN
-F 1 "+3.3V" H 6650 2290 50  0000 C CNN
-F 2 "" H 6650 2150 50  0000 C CNN
-F 3 "" H 6650 2150 50  0000 C CNN
-	1    6650 2150
-	1    0    0    -1
-$EndComp
-$Comp
-L +3.3V #PWR?
+P 6650 2550
+F 0 "#PWR04" H 6650 2400 50  0001 C CNN
+F 1 "+3.3V" H 6650 2690 50  0000 C CNN
+F 2 "" H 6650 2550 50  0000 C CNN
+F 3 "" H 6650 2550 50  0000 C CNN
+	1    6650 2550
+	1    0    0    -1
+$EndComp
+$Comp
+L +3.3V #PWR05
 U 1 1 58D6E79B
 P 9050 2700
-F 0 "#PWR?" H 9050 2550 50  0001 C CNN
+F 0 "#PWR05" H 9050 2550 50  0001 C CNN
 F 1 "+3.3V" H 9050 2840 50  0000 C CNN
 F 2 "" H 9050 2700 50  0000 C CNN
@@
 $EndComp
 $Comp
-L +3.3V #PWR?
+L +3.3V #PWR06
 U 1 1 58D6E7CF
 P 9350 2700
-F 0 "#PWR?" H 9350 2550 50  0001 C CNN
+F 0 "#PWR06" H 9350 2550 50  0001 C CNN
 F 1 "+3.3V" H 9350 2840 50  0000 C CNN
 F 2 "" H 9350 2700 50  0000 C CNN
@@
 $EndComp
 $Comp
-L +3.3V #PWR?
+L +3.3V #PWR07
 U 1 1 58D6E803
-P 8650 2400
-F 0 "#PWR?" H 8650 2250 50  0001 C CNN
-F 1 "+3.3V" H 8650 2540 50  0000 C CNN
-F 2 "" H 8650 2400 50  0000 C CNN
-F 3 "" H 8650 2400 50  0000 C CNN
-	1    8650 2400
-	1    0    0    -1
-$EndComp
-Wire Wire Line
-	8650 2400 8650 3050
+P 8650 2700
+F 0 "#PWR07" H 8650 2550 50  0001 C CNN
+F 1 "+3.3V" H 8650 2840 50  0000 C CNN
+F 2 "" H 8650 2700 50  0000 C CNN
+F 3 "" H 8650 2700 50  0000 C CNN
+	1    8650 2700
+	1    0    0    -1
+$EndComp
+Wire Wire Line
+	8650 2700 8650 3050
 Wire Wire Line
 	9350 2700 9350 2800
@@
 	6750 3150 6200 3150
 $Comp
-L GND #PWR?
+L GND #PWR08
 U 1 1 58D6ED20
 P 6200 4200
-F 0 "#PWR?" H 6200 3950 50  0001 C CNN
+F 0 "#PWR08" H 6200 3950 50  0001 C CNN
 F 1 "GND" H 6200 4050 50  0000 C CNN
 F 2 "" H 6200 4200 50  0000 C CNN
@@
 	6200 4100 6200 4200
 $Comp
-L GND #PWR?
+L GND #PWR09
 U 1 1 58D6F166
 P 2850 4050
-F 0 "#PWR?" H 2850 3800 50  0001 C CNN
+F 0 "#PWR09" H 2850 3800 50  0001 C CNN
 F 1 "GND" H 2850 3900 50  0000 C CNN
 F 2 "" H 2850 4050 50  0000 C CNN
@@
 $EndComp
 $Comp
-L GND #PWR?
+L GND #PWR010
 U 1 1 58D6F261
 P 4850 4250
-F 0 "#PWR?" H 4850 4000 50  0001 C CNN
+F 0 "#PWR010" H 4850 4000 50  0001 C CNN
 F 1 "GND" H 4850 4100 50  0000 C CNN
 F 2 "" H 4850 4250 50  0000 C CNN
@@
 	4850 4150 4850 4250
 $Comp
-L GND #PWR?
+L GND #PWR011
 U 1 1 58D6F42E
 P 6000 3150
-F 0 "#PWR?" H 6000 2900 50  0001 C CNN
+F 0 "#PWR011" H 6000 2900 50  0001 C CNN
 F 1 "GND" H 6000 3000 50  0000 C CNN
 F 2 "" H 6000 3150 50  0000 C CNN
@@
 $EndComp
 $Comp
-L GND #PWR?
+L GND #PWR012
 U 1 1 58D6F4C6
 P 5200 4550
-F 0 "#PWR?" H 5200 4300 50  0001 C CNN
+F 0 "#PWR012" H 5200 4300 50  0001 C CNN
 F 1 "GND" H 5200 4400 50  0000 C CNN
 F 2 "" H 5200 4550 50  0000 C CNN
@@
 	5350 4550 5200 4550
 $Comp
-L GND #PWR?
+L GND #PWR013
 U 1 1 58D6F646
 P 6900 4550
-F 0 "#PWR?" H 6900 4300 50  0001 C CNN
+F 0 "#PWR013" H 6900 4300 50  0001 C CNN
 F 1 "GND" H 6900 4400 50  0000 C CNN
 F 2 "" H 6900 4550 50  0000 C CNN
@@
 	6900 4450 6900 4550
 $Comp
-L GND #PWR?
-U 1 1 58D75EF7
-P 8850 4800
-F 0 "#PWR?" H 8850 4550 50  0001 C CNN
-F 1 "GND" H 8850 4650 50  0000 C CNN
-F 2 "" H 8850 4800 50  0000 C CNN
-F 3 "" H 8850 4800 50  0000 C CNN
-	1    8850 4800
-	1    0    0    -1
-$EndComp
-$Comp
-L GND #PWR?
-U 1 1 58D75F4F
-P 10050 4900
-F 0 "#PWR?" H 10050 4650 50  0001 C CNN
-F 1 "GND" H 10050 4750 50  0000 C CNN
-F 2 "" H 10050 4900 50  0000 C CNN
-F 3 "" H 10050 4900 50  0000 C CNN
-	1    10050 4900
-	1    0    0    -1
-$EndComp
-Wire Wire Line
-	9950 4800 10050 4800
-Wire Wire Line
-	10050 4800 10050 4900
-Wire Wire Line
-	9050 4700 8850 4700
-Wire Wire Line
-	8850 4700 8850 4800
-$Comp
-L R R3
-U 1 1 58D856A4
-P 6650 2400
-F 0 "R3" V 6730 2400 50  0000 C CNN
-F 1 "0" V 6650 2400 50  0000 C CNN
-F 2 "Resistors_SMD:R_0805_HandSoldering" H 6550 3000 50  0000 C CNN
-F 3 "" H 6650 2400 50  0000 C CNN
-	1    6650 2400
-	1    0    0    -1
-$EndComp
-Wire Wire Line
-	6650 2150 6650 2250
+L SF303GJ26 U5
+U 1 1 59534F8F
+P 9650 4850
+F 0 "U5" H 9500 4900 60  0000 C CNN
+F 1 "SF303GJ26" H 9500 5150 60  0000 C CNN
+F 2 "SF303GJ26:SF303GJ26" H 9450 4500 60  0000 C CNN
+F 3 "" H 9650 4850 60  0000 C CNN
+	1    9650 4850
+	1    0    0    -1
+$EndComp
+$Comp
+L GND #PWR014
+U 1 1 5953540A
+P 10100 5000
+F 0 "#PWR014" H 10100 4750 50  0001 C CNN
+F 1 "GND" H 10100 4850 50  0000 C CNN
+F 2 "" H 10100 5000 50  0000 C CNN
+F 3 "" H 10100 5000 50  0000 C CNN
+	1    10100 5000
+	1    0    0    -1
+$EndComp
+Wire Wire Line
+	10000 4800 10100 4800
+Wire Wire Line
+	10100 4800 10100 5000
+Wire Wire Line
+	6650 2550 6650 2650
+Connection ~ 6000 3050
+$Comp
+L CONN_01X02 P5
+U 1 1 5955C1D8
+P 6050 2650
+F 0 "P5" H 6050 2800 50  0000 C CNN
+F 1 "PROGRAM" V 6200 2650 50  0000 C CNN
+F 2 "Pin_Headers:Pin_Header_Straight_1x02_Pitch2.00mm" V 6550 2650 50  0000 C CNN
+F 3 "" H 6050 2650 50  0000 C CNN
+	1    6050 2650
+	0    -1   -1   0
+$EndComp
+NoConn ~ 7700 2550
+NoConn ~ 9000 4800
+Wire Wire Line
+	10000 4900 10200 4900
+Wire Wire Line
+	10200 4900 10200 3150
+Wire Wire Line
+	10200 3150 8550 3150
+Wire Wire Line
+	10000 4700 10100 4700
+Wire Wire Line
+	10100 4700 10100 3250
+Wire Wire Line
+	10100 3250 8550 3250
+Wire Wire Line
+	9000 4900 8900 4900
+Wire Wire Line
+	8900 4900 8900 3350
+Wire Wire Line
+	8900 3350 8550 3350
+Wire Wire Line
+	9000 4700 8800 4700
+Wire Wire Line
+	8800 4700 8800 3450
+Wire Wire Line
+	8800 3450 8550 3450
 $EndSCHEMATC

Commit message: v2.7 of the coordinator board
Parts:
- removed P5: PROGRAM, Pin_Headers:Pin_Header_Straight_1x02_Pitch2.00mm, symbol CONN_01X02
- added R7, R8: 0, Resistors_SMD:R_0805_HandSoldering, symbol R
- added RP1: 10k, R_Array:R_Array_Concave_4x0805, symbol R_PACK4
- added SW2: Switch_DPST, KMR6:KMR641NG, symbol Switch_DPST
Connections:
- net +3V3: now also RP1.5 (R4), RP1.6 (R3), RP1.7 (R2), RP1.8 (R1)
- net GND: now also SW2.4
- net at R2.1, U3.12 (GPIO0): now also SW2.3
- net at U3.4 (GPIO16), U5.1 (A): now also RP1.1 (P1)
- net at U3.5 (GPIO14), U5.3 (C): now also RP1.2 (P2)
- net at U3.6 (GPIO12), U5.4 (B): now also RP1.3 (P3)
- net at U3.7 (GPIO13): now also R7.1, R8.1, RP1.4 (P4); no longer U5.6 (D)
- net at U5.2 (BTN): now also R8.2
- new net: R7.2, U5.6 (D)
- no-connect marks 8 -> 9
Changed lines of the file:
@@
 	6650 2950 6650 3350
 Wire Wire Line
-	6000 2850 6000 3150
-Wire Wire Line
-	6100 2850 6100 3350
+	6000 3050 6000 3150
+Wire Wire Line
+	6100 2750 6100 3350
 Connection ~ 6650 3350
 Wire Wire Line
@@
 F 0 "R6" V 9430 2950 50  0000 C CNN
 F 1 "10k" V 9350 2950 50  0000 C CNN
-F 2 "Resistors_SMD:R_0805_HandSoldering" V 9550 3300 50  0000 C CNN
+F 2 "Resistors_SMD:R_0805_HandSoldering" V 9600 3150 50  0000 C CNN
 F 3 "" H 9350 2950 50  0000 C CNN
 	1    9350 2950
@@
 P 9650 4850
 F 0 "U5" H 9500 4900 60  0000 C CNN
-F 1 "SF303GJ26" H 9500 5150 60  0000 C CNN
+F 1 "SF303GJ26" H 9500 4650 60  0000 C CNN
 F 2 "SF303GJ26:SF303GJ26" H 9450 4500 60  0000 C CNN
 F 3 "" H 9650 4850 60  0000 C CNN
@@
 Wire Wire Line
 	6650 2550 6650 2650
-Connection ~ 6000 3050
-$Comp
-L CONN_01X02 P5
-U 1 1 5955C1D8
-P 6050 2650
-F 0 "P5" H 6050 2800 50  0000 C CNN
-F 1 "PROGRAM" V 6200 2650 50  0000 C CNN
-F 2 "Pin_Headers:Pin_Header_Straight_1x02_Pitch2.00mm" V 6550 2650 50  0000 C CNN
-F 3 "" H 6050 2650 50  0000 C CNN
-	1    6050 2650
+NoConn ~ 7700 2550
+Wire Wire Line
+	10100 3250 10100 4700
+Wire Wire Line
+	10100 3250 8550 3250
+Wire Wire Line
+	8900 4900 9000 4900
+Wire Wire Line
+	8900 3350 8900 4900
+Wire Wire Line
+	8900 3350 8550 3350
+Wire Wire Line
+	8800 4700 9000 4700
+Wire Wire Line
+	8800 3450 8550 3450
+$Comp
+L Switch_DPST SW2
+U 1 1 59611BF3
+P 5900 2450
+F 0 "SW2" V 6050 2450 50  0000 C CNN
+F 1 "Switch_DPST" V 5950 1850 50  0000 C CNN
+F 2 "KMR6:KMR641NG" V 6400 2450 50  0000 C CNN
+F 3 "" H 5900 2450 50  0000 C CNN
+	1    5900 2450
+	0    1    -1   0
+$EndComp
+$Comp
+L GND #PWR015
+U 1 1 59615099
+P 6300 2150
+F 0 "#PWR015" H 6300 1900 50  0001 C CNN
+F 1 "GND" H 6300 2000 50  0000 C CNN
+F 2 "" H 6300 2150 50  0000 C CNN
+F 3 "" H 6300 2150 50  0000 C CNN
+	1    6300 2150
+	1    0    0    -1
+$EndComp
+Wire Wire Line
+	6100 2050 6100 2150
+Wire Wire Line
+	6100 2050 6300 2050
+Wire Wire Line
+	6300 2050 6300 2150
+NoConn ~ 5700 2150
+NoConn ~ 5700 2750
+$Comp
+L R_PACK4 RP1
+U 1 1 59615F7B
+P 9650 4200
+F 0 "RP1" H 9650 4650 50  0000 C CNN
+F 1 "10k" H 9650 4150 50  0000 C CNN
+F 2 "R_Array:R_Array_Concave_4x0805" H 10300 3400 50  0000 C CNN
+F 3 "" H 9650 4200 50  0000 C CNN
+	1    9650 4200
 	0    -1   -1   0
 $EndComp
-NoConn ~ 7700 2550
-NoConn ~ 9000 4800
+Wire Wire Line
+	8800 3450 8800 4700
+Wire Wire Line
+	10100 4700 10000 4700
+Wire Wire Line
+	10200 3150 8550 3150
+$Comp
+L +3.3V #PWR016
+U 1 1 59616333
+P 9600 3800
+F 0 "#PWR016" H 9600 3650 50  0001 C CNN
+F 1 "+3.3V" H 9600 3940 50  0000 C CNN
+F 2 "" H 9600 3800 50  0000 C CNN
+F 3 "" H 9600 3800 50  0000 C CNN
+	1    9600 3800
+	1    0    0    -1
+$EndComp
+Wire Wire Line
+	9600 3800 9600 4000
+Wire Wire Line
+	9300 3900 9600 3900
+Wire Wire Line
+	9500 3900 9500 4000
+Connection ~ 9600 3900
+Wire Wire Line
+	9400 3900 9400 4000
+Connection ~ 9500 3900
+Wire Wire Line
+	9300 3900 9300 4000
+Connection ~ 9400 3900
+Wire Wire Line
+	9300 4400 9300 4450
+Wire Wire Line
+	9400 4400 9400 4550
+Connection ~ 8800 4450
+Wire Wire Line
+	9500 4400 9500 4550
+Connection ~ 10200 4450
+Wire Wire Line
+	9600 4400 9600 4450
+Connection ~ 10100 4550
+Connection ~ 8900 4550
+Wire Wire Line
+	9600 4450 10400 4450
+Wire Wire Line
+	9500 4550 10100 4550
+Wire Wire Line
+	9400 4550 8900 4550
+Wire Wire Line
+	9300 4450 8800 4450
+$Comp
+L R R7
+U 1 1 5961DC36
+P 10200 4750
+F 0 "R7" V 10280 4750 50  0000 C CNN
+F 1 "0" V 10200 4750 50  0000 C CNN
+F 2 "Resistors_SMD:R_0805_HandSoldering" V 10130 4750 50  0001 C CNN
+F 3 "" H 10200 4750 50  0001 C CNN
+	1    10200 4750
+	1    0    0    -1
+$EndComp
+$Comp
+L R R8
+U 1 1 5961DC89
+P 10400 4750
+F 0 "R8" V 10480 4750 50  0000 C CNN
+F 1 "0" V 10400 4750 50  0000 C CNN
+F 2 "Resistors_SMD:R_0805_HandSoldering" V 10330 4750 50  0001 C CNN
+F 3 "" H 10400 4750 50  0001 C CNN
+	1    10400 4750
+	1    0    0    -1
+$EndComp
+Wire Wire Line
+	10200 3150 10200 4600
+Wire Wire Line
+	10400 4450 10400 4600
 Wire Wire Line
 	10000 4900 10200 4900
 Wire Wire Line
-	10200 4900 10200 3150
-Wire Wire Line
-	10200 3150 8550 3150
-Wire Wire Line
-	10000 4700 10100 4700
-Wire Wire Line
-	10100 4700 10100 3250
-Wire Wire Line
-	10100 3250 8550 3250
-Wire Wire Line
-	9000 4900 8900 4900
-Wire Wire Line
-	8900 4900 8900 3350
-Wire Wire Line
-	8900 3350 8550 3350
-Wire Wire Line
-	9000 4700 8800 4700
-Wire Wire Line
-	8800 4700 8800 3450
-Wire Wire Line
-	8800 3450 8550 3450
+	9000 4800 8800 4800
+Wire Wire Line
+	8800 4800 8800 5300
+Wire Wire Line
+	8800 5300 10400 5300
+Wire Wire Line
+	10400 5300 10400 4900
 $EndSCHEMATC
