File: coordinator_board/Coordinator Board.kicad_pcb (KiCad board)
At the start: 4 copper layers, 45.5 x 39.6 mm, 30 parts, among them J1 Conn_01x04, J2 Conn_01x04, J3 Conn_01x04, P4 SERIAL, SW1 Switch_SPDT_x2, SW2 Switch_DPST, U0 10118194, U1 LM3671, U2 CD74HC4050, U3 ESP-12E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

Commit message: Tweaked silk screen layout
Other:
- board text added: "FUSE"
- board text added: "STS"
Changed lines of the file:
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@@
     (area 91.8306 95.957314 143.09421 143.0334)
     (thickness 1.6)
-    (drawings 7)
+    (drawings 9)
     (tracks 338)
     (zones 0)
@@
   (layers
     (0 F.Cu signal)
-    (1 Ground.Plane power)
-    (2 Power.Plane power)
+    (1 Ground.Plane power hide)
+    (2 Power.Plane power hide)
     (31 B.Cu signal)
     (32 B.Adhes user)
@@
     (tags "capacitor 0805")
     (attr smd)
-    (fp_text reference C1 (at 3.048 0 180) (layer B.SilkS)
+    (fp_text reference C1 (at 3.302 -0.635 180) (layer B.SilkS)
       (effects (font (size 1 1) (thickness 0.15)) (justify mirror))
     )
@@
       (effects (font (size 1 1) (thickness 0.15)) (justify mirror))
     )
-    (fp_text user %R (at -3.4 0 180) (layer B.SilkS)
+    (fp_text user %R (at -3.175 0.508 180) (layer B.SilkS)
       (effects (font (size 1 1) (thickness 0.15)) (justify mirror))
     )
@@
     (tags "resistor 0805")
     (attr smd)
-    (fp_text reference R4 (at -3.429 0 180) (layer F.SilkS)
+    (fp_text reference R4 (at 3.683 0.127 180) (layer F.SilkS)
       (effects (font (size 1 1) (thickness 0.15)))
     )
@@
     (tags "resistor 0805")
     (attr smd)
-    (fp_text reference R8 (at 3.556 -0.127 90) (layer F.SilkS)
+    (fp_text reference R8 (at -3.175 0 90) (layer F.SilkS)
       (effects (font (size 1 1) (thickness 0.15)))
     )
@@
   (module nebrius-discrete:R_Array_Concave_4x0805 (layer F.Cu)
     (at 109.922 116.114)
-    (fp_text reference RP1 (at -0.127 2.667) (layer F.SilkS)
+    (fp_text reference RP1 (at 1.651 2.794) (layer F.SilkS)
       (effects (font (size 1 1) (thickness 0.15)))
     )
@@
     (tags "SOIC 1.27")
     (attr smd)
-    (fp_text reference U2 (at -0.254 0 180) (layer F.SilkS)
+    (fp_text reference U2 (at -0.254 0 180) (layer F.SilkS) hide
       (effects (font (size 1 1) (thickness 0.15)))
     )
@@
     (tags "SOT-23-6 Handsoldering")
     (attr smd)
-    (fp_text reference U6 (at 3.175 -0.127 180) (layer F.SilkS)
+    (fp_text reference U6 (at 3.175 -0.127 180) (layer F.SilkS) hide
       (effects (font (size 1 1) (thickness 0.15)))
     )
@@
     (tags "SOT-23-6 Handsoldering")
     (attr smd)
-    (fp_text reference U7 (at 3.175 0 180) (layer F.SilkS)
+    (fp_text reference U7 (at 3.175 0 180) (layer F.SilkS) hide
       (effects (font (size 1 1) (thickness 0.15)))
     )
@@
     (tags "resistor 0805")
     (attr smd)
-    (fp_text reference F0 (at 1.27 1.778 270) (layer F.SilkS)
+    (fp_text reference F0 (at 1.27 1.778 270) (layer F.SilkS) hide
       (effects (font (size 1 1) (thickness 0.15)))
     )
@@
   (module nebrius-conn:10118194 (layer F.Cu)
     (at 95.19 124.242 270)
-    (fp_text reference U0 (at 0 -5.08 270) (layer F.SilkS)
+    (fp_text reference U0 (at 0.254 4.826 270) (layer F.SilkS) hide
       (effects (font (size 1 1) (thickness 0.15)))
     )
@@
       (net 4 GND))
   )
+  (gr_text STS (at 137.989 122.21 90) (layer F.SilkS)
+    (effects (font (size 1 1) (thickness 0.15)))
+  )
+  (gr_text FUSE (at 97.73 117.13 90) (layer F.SilkS)
+    (effects (font (size 1 1) (thickness 0.15)))
+  )
   (gr_line (start 139.386 103.16) (end 93.92 103.16) (angle 90) (layer Edge.Cuts) (width 0.1))
   (gr_line (start 139.386 142.784) (end 139.386 103.16) (angle 90) (layer Edge.Cuts) (width 0.1))
@@
     (effects (font (size 1 1) (thickness 0.15)))
   )
-  (gr_text "Raver Lights Coordinator v3.0\nCopyright Bryan Hughes 2018" (at 137.354 114.971 90) (layer B.SilkS)
+  (gr_text "Raver Lights Coordinator v3.0\nCopyright Bryan Hughes 2018" (at 137.481 115.098 270) (layer B.SilkS)
     (effects (font (size 1 1) (thickness 0.15)) (justify mirror))
   )
