File: board/Coordinator Board.sch (KiCad schematic (older format))
At the start: 31 parts, among them J1 Conn_01x04, J2 Conn_01x04, J3 Conn_01x04, P4 SERIAL, SW1 Switch_SPDT_x2, SW2 Switch_DPST, U0 10118194, U1 LM3671, U2 CD74HC4050, U3 ESP-12E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

Commit message: Finished and ordered v3.0 of the board!!
Connections:
- net at RP1.4 (P4), U5.4 (B): now also U3.14 (GPIO5); no longer U3.13 (GPIO4)
- net at RP1.3 (P3), U5.6 (D): now also U3.13 (GPIO4); no longer U3.14 (GPIO5)
- net at R7.2, U3.19 (GPIO9): now also U5.3 (C); no longer U5.1 (A)
- net at RP1.2 (P2), U3.6 (GPIO12): now also U5.1 (A); no longer U5.2 (BTN)
- net at RP1.1 (P1), U3.7 (GPIO13): now also U5.2 (BTN); no longer U5.3 (C)

Commit message: Updated through first build
Parts:
- C3: footprint (none) -> Capacitors_SMD:C_0805_HandSoldering
Other:
- moved on the sheet: C1, C2, C3, C4, C5, C6, D1, F0, J1, J2, J3, L1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

Commit message: Initial 3.1 board redesign
Parts:
- removed C3: 0.1uF, Capacitors_SMD:C_0805_HandSoldering, symbol C
- removed C4, C5, C6: 10uF, Resistors_SMD:R_0805_HandSoldering, symbol C
- removed D1: LED, LEDs:LED_1206_HandSoldering, symbol LED
- removed R1, R4, R7: 10k, Resistors_SMD:R_0805_HandSoldering, symbol R
- removed R8: 0, Resistors_SMD:R_0805_HandSoldering, symbol R
- removed U2: CD74HC4050, Housings_SOIC:SOIC-16W_5.3x10.2mm_Pitch1.27mm, symbol CD74HC4050
- added J3: Conn_01x04, Pin_Headers:Pin_Header_Angled_1x04_Pitch2.54mm, symbol Conn_01x04
- added RV1: POT, nebrius-discrete:Model-35-Pot, symbol POT
- U1: symbol LM3671 -> LM3671-RESCUE-Coordinator_Board
- U6: value SN74LVC1T45 -> SN74LVC1T45 - MOSI
- U7: value SN74LVC1T45 -> SN74LVC1T45 - SCLK
- renumbered J3 to J4
Connections:
- net +3V3: now also RP1.4 (P4), U5.5 (COM), RV1.3; no longer RP1.5 (R4), RP1.6 (R3), RP1.7 (R2), RP1.8 (R1)
- net +5V: now also J3.1 (Pin_1)
- net GND: now also RP1.1 (P1), RP1.2 (P2), RP1.3 (P3), J3.4 (Pin_4), RV1.1; no longer U5.5 (COM)
- net at U3.10 (GPIO15): now also RP1.8 (R1), U5.2 (BTN)
- net at U3.11 (GPIO2): now also RP1.5 (R4)
- net at U5.3 (C): now also RP1.6 (R3), U3.14 (GPIO5); no longer U3.19 (GPIO9)
- net at U3.2 (ADC): now also RV1.2
- net at U3.21 (MOSI): no longer U6.4 (B)
- net at U3.22 (SCLK): no longer U7.4 (B)
- net at U3.4 (GPIO16): now also U4.4 (SDA); no longer U4.3 (SCL)
- net at U3.5 (GPIO14): now also U7.4 (B); no longer U4.4 (SDA)
- net at J1.2 (Pin_2): now also J2.2 (Pin_2), J4.2 (Pin_2), U7.3 (A), J3.2 (Pin_2)
- net at J1.3 (Pin_3): now also J2.3 (Pin_3), J4.3 (Pin_3), U6.3 (A), J3.3 (Pin_3)
- new net: RP1.7 (R2), U3.13 (GPIO4), U5.4 (B)
- new net: U3.6 (GPIO12), U4.3 (SCL)
- new net: U3.7 (GPIO13), U6.4 (B)
- now unconnected: U5.1 (A), U5.6 (D)
- no-connect marks 9 -> 14
Other:
- moved on the sheet: J1, J2, RP1, U4, U5

Commit message: Finished v3.1 of the board
Connections:
- net at RP1.7 (R2), U3.13 (GPIO4): now also U5.6 (D); no longer U5.4 (B)
- net at RP1.6 (R3), U3.14 (GPIO5): now also U5.1 (A); no longer U5.3 (C)
- net at U3.4 (GPIO16): now also U4.3 (SCL); no longer U4.4 (SDA)
- net at U3.6 (GPIO12): now also U4.4 (SDA); no longer U4.3 (SCL)
Other:
- moved on the sheet: J1, J2, J3, J4, U6, U7

Commit message: Updated r array footprint
Parts:
- RP1: footprint nebrius-discrete:R_Array_Concave_4x0805 -> nebrius-discrete:R_Array_Concave_4x2012.kicad_mod
Changed lines of the file:
@@
 F 0 "RP1" H 5550 6800 50  0000 C CNN
 F 1 "10k" H 5550 6300 50  0000 C CNN
-F 2 "nebrius-discrete:R_Array_Concave_4x0805" V 4700 6900 50  0000 C CNN
+F 2 "nebrius-discrete:R_Array_Concave_4x2012.kicad_mod" V 4700 6900 50  0000 C CNN
 F 3 "" H 5550 6350 50  0000 C CNN
 	1    5550 6350
