File: hub_board/Hub Board.kicad_pcb (KiCad board)
At the start: 4 copper layers, 42.5 x 38.5 mm, 23 parts, among them J1 Conn_01x04, J2 Conn_01x04, J3 Conn_01x04, J4 Conn_01x04, P4 SERIAL, SW1 Switch_SPDT_x2, SW2 Switch_DPST, U0 10118194, U1 LM3671, U3 ESP-12E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

Commit message: Finished redesign, third times the charm?
Parts:
- removed R2: 1k, Resistors_SMD:R_0805_HandSoldering
- removed R5, R6: 10k, Resistors_SMD:R_0805_HandSoldering
- removed RV1: POT, nebrius-discrete:Model-35-Pot
- added J5: Sensor, Pin_Headers:Pin_Header_Straight_1x03_Pitch2.00mm, F.Cu at (130.1, 105.2)
- added R1: 1k, Resistors_SMD:R_0805_HandSoldering, F.Cu at (114.1, 118.4)
- added R4: 10k, Resistors_SMD:R_0805_HandSoldering, B.Cu at (122.1, 125.1)
- added R7: 0, Resistors_SMD:R_0805_HandSoldering, B.Cu at (117.3, 125.1)
- added R8: 0, Resistors_SMD:R_0805_HandSoldering, B.Cu at (118.9, 104.0)
- added RP2: 10k, nebrius-discrete:R_Array_Concave_4x2012.kicad_mod, F.Cu at (113.1, 112.8)
- added U2: 74AUP1G14, TO_SOT_Packages_SMD:SOT-23-5_HandSoldering, F.Cu at (119.7, 118.0)
- J1, J2, J3, J4: value Conn_01x04 -> DotStar
- moved P4 18.7 mm to (130.1, 109.6)
- moved U3 15.9 mm to (111.6, 107.1), turned to 270 degrees
- moved RP1 14.0 mm to (123.4, 113.2), turned to 90 degrees
- moved U5 7.37 mm to (131.9, 117.4)
- moved SW2 1.28 mm to (132.3, 126.1)
Connections:
- C2 pad 1: +3V3 -> VCC
- L1 pad 2: +3V3 -> VCC
- RP1 pad 1: GND -> Net-(RP1-Pad1)
- RP1 pad 2: GND -> Net-(RP1-Pad2)
- RP1 pad 3: GND -> Net-(R8-Pad2)
- RP1 pad 4: +3V3 -> Net-(RP1-Pad4)
- RP1 pad 5: Net-(RP1-Pad5) -> VCC
- RP1 pad 6: Net-(RP1-Pad6) -> VCC
- RP1 pad 7: Net-(RP1-Pad7) -> VCC
- RP1 pad 8: Net-(RP1-Pad8) -> VCC
- SW2 pad 3: Net-(R2-Pad1) -> Net-(R1-Pad2)
- U1 pad 4: +3V3 -> VCC
- U3 pad 10: Net-(RP1-Pad8) -> Net-(R4-Pad1)
- U3 pad 11: Net-(RP1-Pad5) -> Net-(RP2-Pad2)
- U3 pad 12: Net-(R2-Pad1) -> Net-(R1-Pad2)
- U3 pad 13: Net-(RP1-Pad7) -> Net-(U3-Pad13)
- U3 pad 14: Net-(RP1-Pad6) -> Net-(U3-Pad14)
- U3 pad 4: Net-(U3-Pad4) -> Net-(R8-Pad1)
- U3 pad 5: Net-(U3-Pad5) -> Net-(RP1-Pad2)
- U3 pad 6: Net-(U3-Pad6) -> Net-(RP1-Pad1)
- U3 pad 7: Net-(U3-Pad7) -> Net-(RP1-Pad4)
- U3 pad 8: +3V3 -> VCC
- U4 pad 1: +3V3 -> VCC
- U4 pad 3: Net-(U3-Pad4) -> Net-(U3-Pad14)
- U4 pad 4: Net-(U3-Pad6) -> Net-(U3-Pad13)
- U5 pad 1: Net-(RP1-Pad6) -> Net-(RP1-Pad2)
- U5 pad 2: Net-(RP1-Pad8) -> Net-(RP1-Pad1)
- U5 pad 3: (no net) -> Net-(RP2-Pad1)
- U5 pad 4: (no net) -> Net-(R8-Pad2)
- U5 pad 5: +3V3 -> GND
- U5 pad 6: Net-(RP1-Pad7) -> Net-(RP1-Pad4)
- U6 pad 4: Net-(U3-Pad7) -> Net-(R1-Pad2)
- U6 pad 6: +3V3 -> VCC
- U7 pad 4: Net-(U3-Pad5) -> Net-(RP2-Pad2)
- U7 pad 6: +3V3 -> VCC
Routing:
- net Net-(R2-Pad1): track 42.3 -> 0.00 mm, vias 1 -> 0
- net Net-(RP1-Pad8): track 41.8 -> 0.00 mm, vias 2 -> 0
- net Net-(RP1-Pad7): track 41.2 -> 0.00 mm, vias 1 -> 0
- net +3V3: track 41.1 -> 0.00 mm, vias 8 -> 0
- net Net-(RP1-Pad6): track 39.5 -> 0.00 mm, vias 1 -> 0
- net VCC: track 0.00 -> 28.3 mm, vias 0 -> 6
- net Net-(RP2-Pad2): track 0.00 -> 26.7 mm, vias 0 -> 2
- net Net-(R1-Pad2): track 0.00 -> 24.4 mm, vias 0 -> 1
- net Net-(U3-Pad7): track 20.8 -> 0.00 mm, vias 1 -> 0
- net Net-(R8-Pad2): track 0.00 -> 20.7 mm, vias 0 -> 1
- net Net-(U3-Pad5): track 20.5 -> 0.00 mm, vias 1 -> 0
- net Net-(RP1-Pad4): track 0.00 -> 20.1 mm, vias 0 -> 1
- net Net-(RP2-Pad1): track 0.00 -> 19.3 mm
- net Net-(RP1-Pad1): track 0.00 -> 18.6 mm, vias 0 -> 1
- net Net-(RP1-Pad2): track 0.00 -> 16.9 mm, vias 0 -> 1
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- added copper zone on Power.Plane, net VCC
- removed copper zone on Power.Plane, net +3V3
Other:
- board text added: "PROGRAM"
- board text added: "SENSOR"

Commit message: Forgot to bump the version number on the silkscreen
Other:
- board text added: "Raver Lights Hub v3.2 Copyright Bryan Hughes 2018"
- board text removed: "Raver Lights Hub v3.1 Copyright Bryan Hughes 2018"
Changed lines of the file:
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@@
     (links 88)
     (no_connects 0)
-    (area 89.4366 96.719314 174.478734 158.778401)
+    (area 89.4366 101.3716 141.57021 143.0334)
     (thickness 1.6)
     (drawings 11)
@@
   )
   (setup
-    (last_trace_width 0.6096)
+    (last_trace_width 0.1524)
     (user_trace_width 0.1524)
     (user_trace_width 0.3048)
@@
     (effects (font (size 1 1) (thickness 0.15)))
   )
-  (gr_text "Raver Lights Hub v3.1\nCopyright Bryan Hughes 2018" (at 134.306 129.576 90) (layer B.SilkS)
+  (gr_text "Raver Lights Hub v3.2\nCopyright Bryan Hughes 2018" (at 134.306 129.576 90) (layer B.SilkS)
     (effects (font (size 1 1) (thickness 0.15)) (justify mirror))
   )
