File: endpoint_board/Endpoint Board.kicad_pcb (KiCad board)
At the start: 2 copper layers, 24.8 x 24.8 mm, 11 parts, among them P1 POWER, P2 LIGHT, P3 ESP, P4 SERIAL, SW1 Switch_SPDT_x2, U1 LM3671

Commit message: First draft of the new receivers
Parts:
- removed P1: POWER, Pin_Headers:Pin_Header_Straight_1x02_Pitch2.00mm
- removed P2: LIGHT, Pin_Headers:Pin_Header_Angled_1x04
- removed P3: ESP, Pin_Headers:Pin_Header_Straight_2x04
- removed PGM: PGRM, Pin_Headers:Pin_Header_Straight_1x02_Pitch2.00mm
- removed RUN: RUN, Pin_Headers:Pin_Header_Straight_1x02_Pitch2.00mm
- added R1: 10k, Resistors_SMD:R_0805_HandSoldering, F.Cu at (142.6, 136.7)
- added R2: 1k, Resistors_SMD:R_0805_HandSoldering, F.Cu at (142.6, 143.6)
- added R3: 10k, Resistors_SMD:R_0805_HandSoldering, F.Cu at (142.6, 140.1)
- added U2: ESP-01, Pin_Headers:Pin_Header_Straight_2x04_Pitch2.54mm, F.Cu at (149.7, 144.7)
- added U3: NeoPixel, Pin_Headers:Pin_Header_Angled_1x03_Pitch2.54mm, F.Cu at (137.9, 143.1)
- added U4: SN74LVC1T45, TO_SOT_Packages_SMD:TSOT-23-6_HandSoldering, F.Cu at (140.8, 132.5)
- SW1: value Switch_SPDT_x2 -> SW_DPST; footprint Pin_Headers:Pin_Header_Straight_1x03 -> nebrius-switch:KMR641NG
- U1: footprint TO_SOT_Packages_SMD:SOT-23-5 -> TO_SOT_Packages_SMD:SOT-23-5_HandSoldering
- moved SW1 24.9 mm to (148.5, 132.3), turned to 180 degrees
- moved L1 11.4 mm to (142.6, 138.6)
- moved U1 11.0 mm to (142.6, 142.1)
- moved C2 9.33 mm to (142.5, 136.1), turned to 0 degrees
- moved C1 5.03 mm to (142.6, 146.2), turned to 0 degrees
Connections:
- net Net-(C2-Pad1) renamed VCC
- C1 pad 1: Net-(C1-Pad1) -> +5V
- C1 pad 2: Net-(C1-Pad2) -> GND
- C2 pad 2: Net-(C1-Pad2) -> GND
- P4 pad 1: Net-(C1-Pad2) -> GND
- SW1 pad 2: Net-(C1-Pad1) -> GND
- U1 pad 1: Net-(C1-Pad1) -> +5V
- U1 pad 2: Net-(C1-Pad2) -> GND
- U1 pad 3: Net-(C1-Pad1) -> +5V
Routing:
- net Net-(C1-Pad2): track 47.5 -> 0.00 mm
- net Net-(C1-Pad1): track 30.8 -> 0.00 mm
- net VCC: track 30.2 -> 9.96 mm, vias 0 -> 4
- net Net-(P2-Pad3): track 19.6 -> 0.00 mm
- net Net-(R3-Pad2): track 0.00 -> 11.3 mm
- net Net-(P3-Pad4): track 11.3 -> 0.00 mm
- net +5V: track 0.00 -> 10.4 mm, vias 0 -> 2
- net Net-(P2-Pad2): track 9.53 -> 0.00 mm
- net GND: track 0.00 -> 8.46 mm, vias 0 -> 5
- net Net-(U3-Pad2): track 0.00 -> 7.83 mm
- net Net-(R1-Pad2): track 0.00 -> 6.97 mm, vias 0 -> 1
- net Net-(P4-Pad2): track 24.2 -> 29.0 mm
- net Net-(R2-Pad2): track 12.2 -> 16.7 mm
- net Net-(P4-Pad3): track 14.7 -> 15.3 mm
- added copper zone on Power.Plane, net +5V
- added copper zone on Ground.Plane, net GND
- added copper zone on Power.Plane, net VCC
Other:
- board size 24.8 x 24.8 mm -> 24.8 x 17.5 mm
- copper layers 2 -> 4
- board text added: "Raver Lights Receiver 3.0 Copyright Bryan Hughes"
- board text removed: "+"
- board text removed: "-"
- board text removed: "Power"
- board text removed: "Power Switch"
- board text removed: "RX"
- board text removed: "Raver Lights Endpoint v1.6 Copyright Bryan Hughes"
- board text removed: "TX"
