File: powered_receiver_board/Powered Receiver Board.kicad_pcb (KiCad board)
At the start: 4 copper layers, 24.3 x 17.5 mm, 13 parts, among them P4 SERIAL, SW1 SW_DPST, U1 LM3671, U2 ESP-01, U3 NeoPixel, U4 SN74LVC1T45

Commit message: Updated project to new KiCAD format
Parts:
- added U5: 10118194, nebrius-conn:10118194, F.Cu at (155.4, 139.4)

Commit message: Final version of the powered receiver board
Parts:
- moved U5 16.9 mm to (141.2, 130.3), turned to 180 degrees
- moved U4 6.74 mm to (147.6, 132.1), turned to 270 degrees
- moved SW1 3.21 mm to (151.2, 132.1), turned to 90 degrees
Routing:
- net Net-(U3-Pad2): track 7.83 -> 24.0 mm
- net +5V: track 3.09 -> 18.4 mm, vias 2 -> 3
- net GND: track 8.72 -> 18.6 mm
- net Net-(P4-Pad3): track 15.3 -> 23.5 mm
- net Net-(R2-Pad2): track 16.8 -> 15.2 mm
- net Net-(R3-Pad2): track 11.3 -> 12.1 mm, vias 0 -> 2
Other:
- board size 24.3 x 17.5 mm -> 25.3 x 18.9 mm
- board text added: "Raver Lights Receiver 3.5 Copyright 2018 Bryan Hughes"
- board text removed: "Raver Lights Receiver 3.0 Copyright 2018 Bryan Hughes"
