File: powered_receiver_board/Powered Receiver Board.sch (KiCad schematic (older format))
At the start: 14 parts, among them P4 SERIAL, SW1 SW_DPST, U1 LM3671, U2 ESP-01, U3 NeoPixel, U4 SN74LVC1T45, U5 10118194

Commit message: Final version of the powered receiver board
Other:
- moved on the sheet: F1, U5
Changed lines of the file:
@@
 	9150 3650 8950 3650
 Connection ~ 8950 3650
-Wire Wire Line
-	3700 3000 3850 3000
 Connection ~ 4000 3000
 Wire Wire Line
@@
 L power:+5V #PWR03
 U 1 1 5AF7418F
-P 3300 2900
-F 0 "#PWR03" H 3300 2750 50  0001 C CNN
-F 1 "+5V" H 3300 3040 50  0000 C CNN
-F 2 "" H 3300 2900 50  0001 C CNN
-F 3 "" H 3300 2900 50  0001 C CNN
-	1    3300 2900
-	1    0    0    -1
-$EndComp
-Wire Wire Line
-	3300 2900 3300 3000
+P 3350 2900
+F 0 "#PWR03" H 3350 2750 50  0001 C CNN
+F 1 "+5V" H 3350 3040 50  0000 C CNN
+F 2 "" H 3350 2900 50  0001 C CNN
+F 3 "" H 3350 2900 50  0001 C CNN
+	1    3350 2900
+	1    0    0    -1
+$EndComp
 $Comp
 L power:GND #PWR04
@@
 L Device:Fuse F1
 U 1 1 5AF9F066
-P 3550 3000
-F 0 "F1" V 3630 3000 50  0000 C CNN
-F 1 "Fuse" V 3475 3000 50  0000 C CNN
-F 2 "Resistors_SMD:R_0805_HandSoldering" V 3480 3000 50  0001 C CNN
-F 3 "" H 3550 3000 50  0001 C CNN
-	1    3550 3000
+P 3600 3000
+F 0 "F1" V 3680 3000 50  0000 C CNN
+F 1 "Fuse" V 3525 3000 50  0000 C CNN
+F 2 "Resistors_SMD:R_0805_HandSoldering" V 3530 3000 50  0001 C CNN
+F 3 "" H 3600 3000 50  0001 C CNN
+	1    3600 3000
 	0    1    1    0
 $EndComp
-Wire Wire Line
-	3300 3000 3400 3000
 Wire Wire Line
 	3850 3100 3850 3000
@@
 L nebrius-conn:10118194 U5
 U 1 1 5C334859
-P 2950 3300
-F 0 "U5" V 2363 3394 60  0000 C CNN
-F 1 "10118194" V 2469 3394 60  0000 C CNN
-F 2 "nebrius-conn:10118194" H 2950 3300 60  0001 C CNN
-F 3 "" H 2950 3300 60  0001 C CNN
-	1    2950 3300
+P 3000 3300
+F 0 "U5" V 2413 3394 60  0000 C CNN
+F 1 "10118194" V 2519 3394 60  0000 C CNN
+F 2 "nebrius-conn:10118194" H 3000 3300 60  0001 C CNN
+F 3 "" H 3000 3300 60  0001 C CNN
+	1    3000 3300
 	0    -1   1    0
 $EndComp
-Wire Wire Line
-	3150 3000 3300 3000
-Connection ~ 3300 3000
 $Comp
 L power:GND #PWR0101
 U 1 1 5C336DF8
-P 3250 3500
-F 0 "#PWR0101" H 3250 3250 50  0001 C CNN
-F 1 "GND" H 3255 3327 50  0000 C CNN
-F 2 "" H 3250 3500 50  0001 C CNN
-F 3 "" H 3250 3500 50  0001 C CNN
-	1    3250 3500
-	1    0    0    -1
-$EndComp
-Wire Wire Line
-	3150 3400 3250 3400
-Wire Wire Line
-	3250 3400 3250 3500
-NoConn ~ 3150 3100
-NoConn ~ 3150 3200
-NoConn ~ 3150 3300
+P 3350 3500
+F 0 "#PWR0101" H 3350 3250 50  0001 C CNN
+F 1 "GND" H 3355 3327 50  0000 C CNN
+F 2 "" H 3350 3500 50  0001 C CNN
+F 3 "" H 3350 3500 50  0001 C CNN
+	1    3350 3500
+	1    0    0    -1
+$EndComp
+Wire Wire Line
+	3200 3400 3350 3400
+Wire Wire Line
+	3350 3400 3350 3500
+NoConn ~ 3200 3100
+NoConn ~ 3200 3200
+NoConn ~ 3200 3300
+Wire Wire Line
+	3450 3000 3350 3000
+Wire Wire Line
+	3750 3000 3850 3000
+Wire Wire Line
+	3350 2900 3350 3000
+Connection ~ 3350 3000
+Wire Wire Line
+	3350 3000 3200 3000
 $EndSCHEMATC
