File: boards/hub/Hub Board.kicad_pcb (KiCad board)
At the start: 4 copper layers, 42.5 x 38.5 mm, 22 parts, among them J1 NeoPixel, J2 NeoPixel, J3 NeoPixel, J4 NeoPixel, J5 Sensor, P4 SERIAL, SW1 Switch_SPDT_x2, SW2 Switch_DPST, U0 10118194, U1 LM3671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

Commit message: More work migrating things to the new version of Kicad
Connections:
- SW1 pad 1: (no net) -> Net-(SW1-Pad1)
- SW2 pad 1: (no net) -> Net-(SW2-Pad1)
- SW2 pad 2: (no net) -> Net-(SW2-Pad2)
- U0 pad 2: (no net) -> Net-(U0-Pad2)
- U0 pad 3: (no net) -> Net-(U0-Pad3)
- U0 pad 4: (no net) -> Net-(U0-Pad4)
- U3 pad 17: (no net) -> Net-(U3-Pad17)
- U3 pad 18: (no net) -> Net-(U3-Pad18)
- U3 pad 19: (no net) -> Net-(U3-Pad19)
- U3 pad 20: (no net) -> Net-(U3-Pad20)
- U3 pad 21: (no net) -> Net-(U3-Pad21)
- U3 pad 22: (no net) -> Net-(U3-Pad22)
