File: boards/hub/Hub Board.sch (KiCad schematic (older format))
At the start: 22 parts, among them J1 NeoPixel, J2 NeoPixel, J3 NeoPixel, J4 NeoPixel, J5 Sensor, P4 SERIAL, SW1 Switch_SPDT_x2, SW2 Switch_DPST, U0 10118194, U1 LM3671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

Commit message: More work migrating things to the new version of Kicad
Parts:
- C1, C2: symbol C -> Hub-Board-rescue:C
- F0: symbol Fuse -> Hub-Board-rescue:Fuse
- J1, J2, J3, J4: symbol NeoPixel -> Hub-Board-rescue:NeoPixel
- J5: symbol Conn_01x03 -> Hub-Board-rescue:Conn_01x03
- L1: symbol INDUCTOR -> Hub-Board-rescue:INDUCTOR
- P4: symbol CONN_01X03 -> Hub-Board-rescue:CONN_01X03
- R1: symbol R -> Hub-Board-rescue:R
- RP1, RP2: symbol R_PACK4 -> Hub-Board-rescue:R_PACK4
- SW1: symbol Switch_SPDT_x2 -> Hub-Board-rescue:Switch_SPDT_x2
- SW2: symbol Switch_DPST -> Hub-Board-rescue:Switch_DPST
- U0: symbol 10118194 -> Hub-Board-rescue:10118194
- U1: symbol LM3671 -> Hub-Board-rescue:LM3671
- U2: symbol 74AUP1G14 -> Hub-Board-rescue:74AUP1G14
- U3: symbol ESP-12E -> Hub-Board-rescue:ESP-12E
- U4: symbol DIY-OLED-0.96 -> Hub-Board-rescue:DIY-OLED-0.96
- U5: symbol SF303GJ26 -> Hub-Board-rescue:SF303GJ26
- U7: symbol SN74LVC1T45 -> Hub-Board-rescue:SN74LVC1T45
