File: boards/configurable_receiver/Configurable Receiver Board.sch (KiCad schematic (older format))
At the start: 18 parts, among them J4 NeoPixel, J5 Sensor, P4 SERIAL, SW1 Switch_SPDT_x2, SW2 Switch_DPST, U0 10118194, U1 LM3671, U3 ESP-12E, U7 SN74LVC1T45

Commit message: More work migrating things to the new version of Kicad
Parts:
- removed J5: Sensor, Pin_Headers:Pin_Header_Straight_1x03_Pitch2.00mm, symbol Configurable-Receiver-Board-rescue:Conn_01x03
- removed SW?: SW_DIP_x02, symbol Switch:SW_DIP_x02
- removed SW?: SW_DIP_x03, symbol Switch:SW_DIP_x03
- added D1, D2: LED, Resistors_SMD:R_0805_HandSoldering, symbol Device:LED
- added R2, R3: 68, Resistors_SMD:R_0805_HandSoldering, symbol Configurable-Receiver-Board-rescue:R
- added RV1: R_POT, symbol Device:R_POT
- added SW?: SW_DIP_x04, symbol Switch:SW_DIP_x04
- gave numbers to parts that had none: 1
Connections:
- wire segments 88 -> 131
Other:
- moved on the sheet: R1, RP1

Commit message: Created v4 of the receiver
Parts:
- removed U3: ESP-12E, ESP8266:ESP-12E_SMD, symbol Configurable-Receiver-Board-rescue:ESP-12E
- added U3: ESP-12F, ESP8266:ESP-12F_SMD, symbol Configurable-Receiver-Board-rescue:ESP-12F
- D1, D2, F0, R1, R2, R3: footprint Resistors_SMD:R_0805_HandSoldering -> Resistor_SMD:R_0805_2012Metric_Pad1.15x1.40mm_HandSolder
- RV1: footprint (none) -> nebrius-switch:TC33-potentiometer
- SW1: footprint CL-SA-12C:CL-SA-12C4 -> nebrius-switch:CL-SA-12C4
- SW3: renamed from SW?; footprint (none) -> Package_DIP:SMDIP-8_W9.53mm
Connections:
- net GND: now also U3.9 (GND)
- net VCC: now also U3.8 (VCC)
- net at P4.1 (P1): now also U3.15 (RXD)
- net at P4.2 (P2): now also U3.16 (TXD)
- net at RP2.4 (P4): now also U3.1 (REST)
- net at RP2.1 (P1): now also U3.10 (GPIO15)
- net at RP2.2 (P2), U7.4 (B): now also U3.11 (GPIO2)
- net at R1.2, SW2.3: now also U3.12 (GPIO0)
- net at D1.2 (A): now also U3.13 (GPIO4)
- net at D2.2 (A): now also U3.14 (GPIO5)
- net at RV1.2: now also U3.2 (ADC)
- net at RP2.3 (P3): now also U3.3 (CH_PD)
- net at RP1.1 (P1), SW3.4: now also U3.4 (GPIO16)
- net at RP1.2 (P2), SW3.3: now also U3.5 (GPIO14)
- net at RP1.3 (P3), SW3.2: now also U3.6 (GPIO12)
- net at RP1.4 (P4), SW3.1: now also U3.7 (GPIO13)
Changed lines of the file:
@@
 F 0 "SW1" H 2350 4300 50  0000 C CNN
 F 1 "Switch_SPDT_x2" H 2300 4000 50  0000 C CNN
-F 2 "CL-SA-12C:CL-SA-12C4" H 2850 4450 50  0000 C CNN
+F 2 "nebrius-switch:CL-SA-12C4" H 2850 4450 50  0000 C CNN
 F 3 "" H 2550 4150 50  0000 C CNN
 	1    2550 4150
@@
 $EndComp
 $Comp
-L Configurable-Receiver-Board-rescue:ESP-12E U3
-U 1 1 58977E50
-P 6650 4650
-F 0 "U3" H 6650 4550 50  0000 C CNN
-F 1 "ESP-12E" H 6650 4750 50  0000 C CNN
-F 2 "ESP8266:ESP-12E_SMD" H 6650 4650 50  0001 C CNN
-F 3 "" H 6650 4650 50  0001 C CNN
-	1    6650 4650
-	-1   0    0    1
-$EndComp
-$Comp
 L Configurable-Receiver-Board-rescue:GND #PWR01
 U 1 1 58D6F166
@@
 F 0 "F0" V 1530 5200 50  0000 C CNN
 F 1 "Fuse" V 1375 5200 50  0000 C CNN
-F 2 "Resistors_SMD:R_0805_HandSoldering" V 1380 5200 50  0001 C CNN
+F 2 "Resistor_SMD:R_0805_2012Metric_Pad1.15x1.40mm_HandSolder" V 1380 5200 50  0001 C CNN
 F 3 "" H 1450 5200 50  0001 C CNN
 	1    1450 5200
@@
 F 0 "R1" V 5480 4000 50  0000 C CNN
 F 1 "1k" V 5400 4000 50  0000 C CNN
-F 2 "Resistors_SMD:R_0805_HandSoldering" V 5330 4000 50  0001 C CNN
+F 2 "Resistor_SMD:R_0805_2012Metric_Pad1.15x1.40mm_HandSolder" V 5330 4000 50  0001 C CNN
 F 3 "" H 5400 4000 50  0001 C CNN
 	1    5400 4000
@@
 F 0 "RV1" H 9480 4804 50  0000 R CNN
 F 1 "R_POT" H 9480 4895 50  0000 R CNN
-F 2 "" H 9550 4850 50  0001 C CNN
+F 2 "nebrius-switch:TC33-potentiometer" H 9550 4850 50  0001 C CNN
 F 3 "~" H 9550 4850 50  0001 C CNN
 	1    9550 4850
@@
 F 0 "D1" V 5339 5383 50  0000 R CNN
 F 1 "LED" V 5248 5383 50  0000 R CNN
-F 2 "Resistors_SMD:R_0805_HandSoldering" H 5300 5500 50  0001 C CNN
+F 2 "Resistor_SMD:R_0805_2012Metric_Pad1.15x1.40mm_HandSolder" H 5300 5500 50  0001 C CNN
 F 3 "~" H 5300 5500 50  0001 C CNN
 	1    5300 5500
@@
 F 0 "D2" V 5689 5383 50  0000 R CNN
 F 1 "LED" V 5598 5383 50  0000 R CNN
-F 2 "Resistors_SMD:R_0805_HandSoldering" H 5650 5500 50  0001 C CNN
+F 2 "Resistor_SMD:R_0805_2012Metric_Pad1.15x1.40mm_HandSolder" H 5650 5500 50  0001 C CNN
 F 3 "~" H 5650 5500 50  0001 C CNN
 	1    5650 5500
@@
 F 0 "R2" H 5370 5946 50  0000 L CNN
 F 1 "68" V 5300 5850 50  0000 L CNN
-F 2 "Resistors_SMD:R_0805_HandSoldering" V 5230 5900 50  0001 C CNN
+F 2 "Resistor_SMD:R_0805_2012Metric_Pad1.15x1.40mm_HandSolder" V 5230 5900 50  0001 C CNN
 F 3 "" H 5300 5900 50  0001 C CNN
 	1    5300 5900
@@
 F 0 "R3" H 5720 5946 50  0000 L CNN
 F 1 "68" V 5650 5850 50  0000 L CNN
-F 2 "Resistors_SMD:R_0805_HandSoldering" V 5580 5900 50  0001 C CNN
+F 2 "Resistor_SMD:R_0805_2012Metric_Pad1.15x1.40mm_HandSolder" V 5580 5900 50  0001 C CNN
 F 3 "" H 5650 5900 50  0001 C CNN
 	1    5650 5900
@@
 Connection ~ 8550 5250
 $Comp
-L Switch:SW_DIP_x04 SW?
+L Switch:SW_DIP_x04 SW3
 U 1 1 5D0FDBCE
 P 7750 5850
-F 0 "SW?" V 7704 6180 50  0000 L CNN
+F 0 "SW3" V 7704 6180 50  0000 L CNN
 F 1 "SW_DIP_x04" V 7795 6180 50  0000 L CNN
-F 2 "" H 7750 5850 50  0001 C CNN
+F 2 "Package_DIP:SMDIP-8_W9.53mm" H 7750 5850 50  0001 C CNN
 F 3 "~" H 7750 5850 50  0001 C CNN
 	1    7750 5850
@@
 Wire Wire Line
 	7650 6250 7750 6250
+$Comp
+L Configurable-Receiver-Board-rescue:ESP-12F U3
+U 1 1 5CFB0A81
+P 6650 4650
+F 0 "U3" H 6650 3885 50  0000 C CNN
+F 1 "ESP-12F" H 6650 3976 50  0000 C CNN
+F 2 "ESP8266:ESP-12F_SMD" H 6650 4650 50  0001 C CNN
+F 3 "" H 6650 4650 50  0001 C CNN
+	1    6650 4650
+	-1   0    0    1
+$EndComp
 $EndSCHEMATC

Commit message: Started designing next version of the receiver boards
Parts:
- removed RV1: R_POT, nebrius-switch:TC33-potentiometer, symbol Device:R_POT
- removed SW3: SW_DIP_x04, Package_DIP:SMDIP-8_W9.53mm, symbol Switch:SW_DIP_x04
- added P1: SENSOR, Connector_PinHeader_2.00mm:PinHeader_1x03_P2.00mm_Vertical, symbol Configurable-Receiver-Board-rescue:CONN_01X03
- added R4: 0, Resistor_SMD:R_0805_2012Metric_Pad1.15x1.40mm_HandSolder, symbol Configurable-Receiver-Board-rescue:R
- added SW3: SW_DIP_x03, Package_DIP:SMDIP-6_W9.53mm, symbol Switch:SW_DIP_x03
- C1, C2: footprint Capacitors_SMD:C_0805_HandSoldering -> Capacitor_SMD:C_0805_2012Metric_Pad1.15x1.40mm_HandSolder
- L1: footprint Resistors_SMD:R_0805_HandSoldering -> Resistor_SMD:R_0805_2012Metric_Pad1.15x1.40mm_HandSolder
- P4: footprint Pin_Headers:Pin_Header_Straight_1x03_Pitch2.00mm -> Connector_PinHeader_2.00mm:PinHeader_1x03_P2.00mm_Vertical
Connections:
- net GND: now also P1.3 (P3)
- net VCC: now also P1.1 (P1), R4.1, SW3.4, SW3.5, SW3.6
- net at RP1.1 (P1), U3.4 (GPIO16): now also SW3.3
- net at RP1.2 (P2), U3.5 (GPIO14): now also SW3.2
- net at RP1.3 (P3), U3.6 (GPIO12): now also SW3.1
- net at RP1.4 (P4), U3.7 (GPIO13): now also R4.2
- net at U3.2 (ADC): now also P1.2 (P2)
- no-connect marks 12 -> 6
Other:
- moved on the sheet: J4, RP1

Commit message: Finished v4.5 of the receiver board
Connections:
- net at RP1.1 (P1), SW3.3: now also U3.6 (GPIO12); no longer U3.4 (GPIO16)
- net at RP1.3 (P3), SW3.1: now also U3.4 (GPIO16); no longer U3.6 (GPIO12)
Changed lines of the file:
@@
-$EndComp
-$Comp
-L Configurable-Receiver-Board-rescue:+5V #PWR08
-U 1 1 5A47E6D7
-P 8150 2400
-F 0 "#PWR08" H 8150 2250 50  0001 C CNN
-F 1 "+5V" H 8150 2540 50  0000 C CNN
-F 2 "" H 8150 2400 50  0001 C CNN
-F 3 "" H 8150 2400 50  0001 C CNN
-	1    8150 2400
-	1    0    0    -1
 $EndComp
 $Comp
@@
 	7750 4550 7550 4550
 Wire Wire Line
-	7550 4450 7850 4450
-Wire Wire Line
-	7850 4450 7850 5450
-Wire Wire Line
 	7550 4350 7950 4350
 Wire Wire Line
@@
 	5650 6050 5650 6150
 Wire Wire Line
-	7550 4650 7650 4650
-Wire Wire Line
-	7650 4650 7650 5250
-Wire Wire Line
 	7650 5250 7650 5550
 Connection ~ 7650 5250
@@
 Wire Wire Line
 	9500 4950 9500 5050
+$Comp
+L Configurable-Receiver-Board-rescue:+5V #PWR08
+U 1 1 5A47E6D7
+P 8150 2400
+F 0 "#PWR08" H 8150 2250 50  0001 C CNN
+F 1 "+5V" H 8150 2540 50  0000 C CNN
+F 2 "" H 8150 2400 50  0001 C CNN
+F 3 "" H 8150 2400 50  0001 C CNN
+	1    8150 2400
+	1    0    0    -1
+$EndComp
+Wire Wire Line
+	7650 4450 7550 4450
+Wire Wire Line
+	7650 4450 7650 5250
+Wire Wire Line
+	7550 4650 7850 4650
+Wire Wire Line
+	7850 4650 7850 5450
 $EndSCHEMATC
